Commit message: Change resolution and FOV of D435 camera

File: realsense2_description/urdf/_d435.gazebo.xacro (robot description, xacro)
@@ -91,8 +91,9 @@
       <sensor name="${camera_name}depth" type="depth">
         <camera name="${camera_name}">
-          <horizontal_fov>${85.2*deg_to_rad}</horizontal_fov>
+          <!-- <horizontal_fov>${85.2*deg_to_rad}</horizontal_fov> -->
+          <horizontal_fov>${69.4*deg_to_rad}</horizontal_fov>
           <image>
-            <width>1280</width>
-            <height>720</height>
+            <width>640</width>
+            <height>480</height>
           </image>
           <clip>
@@ -107,6 +108,7 @@
         </camera>
         <always_on>1</always_on>
-        <update_rate>90</update_rate>
+        <update_rate>30</update_rate>
         <visualize>0</visualize>
+        <topic>/test/image_raw</topic>
       </sensor>
     </gazebo>

File: realsense2_description/urdf/_d435.urdf.xacro (robot description, xacro)
@@ -16,5 +16,6 @@
     <xacro:property name="d435_cam_depth_to_infra1_offset" value="0.0"/>
     <xacro:property name="d435_cam_depth_to_infra2_offset" value="-0.050"/>
-    <xacro:property name="d435_cam_depth_to_color_offset" value="0.015"/>
+    <!-- <xacro:property name="d435_cam_depth_to_color_offset" value="0.015"/> -->
+    <xacro:property name="d435_cam_depth_to_color_offset" value="0"/>
     <!-- The following values model the aluminum peripherial case for the
   	D435 camera, with the camera joint represented by the actual
